Commit message: UPDATE: moveit works!

File: src/moveit_config/config/moveit_config.ros2_control.xacro (robot description, xacro)
@@ -3,13 +3,12 @@
   <xacro:macro name="motor_drive">
     <ros2_control name="motor_drive" type="system">
-      <!-- <hardware>
+      <hardware>
         <plugin>ethercat_driver/EthercatDriver</plugin>
         <param name="master_id">0</param>
         <param name="control_frequency">100</param>
+      </hardware>
+      <!-- <hardware>
+        <plugin>mock_components/GenericSystem</plugin>
       </hardware> -->
-      <hardware>
-        <!-- By default, set up controllers for simulation. This won't work on real hardware -->
-        <plugin>mock_components/GenericSystem</plugin>
-      </hardware>
       <joint name="joint2">
         <state_interface name="position"/>
@@ -23,6 +22,6 @@
           <param name="alias">0</param>
           <param name="position">0</param>
-          <param name="mode_of_operation">8</param>
-          <param name="slave_config">$(find ethercat_motor_drive)/config/tech_driver.yaml</param>
+          <param name="mode_of_operation">9</param>
+          <param name="slave_config">$(find moveit_config)/driver_config/tech_driver.yaml</param>
         </ec_module>
       </joint>
@@ -38,6 +37,6 @@
           <param name="alias">0</param>
           <param name="position">1</param>
-          <param name="mode_of_operation">8</param>
-          <param name="slave_config">$(find ethercat_motor_drive)/config/tech_driver.yaml</param>
+          <param name="mode_of_operation">9</param>
+          <param name="slave_config">$(find moveit_config)/driver_config/tech_driver.yaml</param>
         </ec_module>
       </joint>
@@ -53,6 +52,6 @@
           <param name="alias">0</param>
           <param name="position">2</param>
-          <param name="mode_of_operation">8</param>
-          <param name="slave_config">$(find ethercat_motor_drive)/config/tech_driver.yaml</param>
+          <param name="mode_of_operation">9</param>
+          <param name="slave_config">$(find moveit_config)/driver_config/tech_driver.yaml</param>
         </ec_module>
       </joint>
@@ -68,6 +67,6 @@
           <param name="alias">0</param>
           <param name="position">3</param>
-          <param name="mode_of_operation">8</param>
-          <param name="slave_config">$(find ethercat_motor_drive)/config/tech_driver.yaml</param>
+          <param name="mode_of_operation">9</param>
+          <param name="slave_config">$(find moveit_config)/driver_config/tech_driver.yaml</param>
         </ec_module>
       </joint>
@@ -83,6 +82,6 @@
           <param name="alias">0</param>
           <param name="position">4</param>
-          <param name="mode_of_operation">8</param>
-          <param name="slave_config">$(find ethercat_motor_drive)/config/tech_driver.yaml</param>
+          <param name="mode_of_operation">9</param>
+          <param name="slave_config">$(find moveit_config)/driver_config/tech_driver.yaml</param>
         </ec_module>
       </joint> -->

File: src/moveit_config/config/robot_description.urdf.xacro (robot description, xacro)
@@ -1,7 +1,7 @@
 <?xml version="1.0"?>
 <robot xmlns:xacro="http://www.ros.org/wiki/xacro">
-  <xacro:macro name="TechRobot">
+  <xacro:macro name="auto_store_manipulator">
   <!-- helper macro -->
-  <xacro:include filename="$(find ethercat_motor_drive)/description/urdf/create_link.xacro"/>
+  <xacro:include filename="$(find moveit_config)/config/create_link.xacro"/>
   <xacro:create_link
       link_name="base_link"
@@ -9,5 +9,5 @@
       rpy_offset="0 0 0"
       mass="23.3444937848516"
-      mesh_path="package://ethercat_motor_drive/meshes"
+      mesh_path="package://moveit_config/meshes"
   />
   <xacro:create_link
@@ -16,5 +16,5 @@
       rpy_offset="0 0 0"
       mass="8.67027571199243"
-      mesh_path="package://ethercat_motor_drive/meshes"
+      mesh_path="package://moveit_config/meshes"
   />
   <xacro:create_link
@@ -23,5 +23,5 @@
       rpy_offset="0 0 0"
       mass="0.647403062770475"
-      mesh_path="package://ethercat_motor_drive/meshes"
+      mesh_path="package://moveit_config/meshes"
   />
   <xacro:create_link
@@ -30,5 +30,5 @@
       rpy_offset="0 0 0"
       mass="0.647403062770475"
-      mesh_path="package://ethercat_motor_drive/meshes"
+      mesh_path="package://moveit_config/meshes"
   />
   <xacro:create_link
@@ -37,5 +37,5 @@
       rpy_offset="0 0 0"
       mass="0.441881459418396"
-      mesh_path="package://ethercat_motor_drive/meshes"
+      mesh_path="package://moveit_config/meshes"
   />
   <xacro:create_link
@@ -44,5 +44,5 @@
       rpy_offset="0 0 0"
       mass="0.359995634810237"
-      mesh_path="package://ethercat_motor_drive/meshes"
+      mesh_path="package://moveit_config/meshes"
   />
   <xacro:create_link
@@ -51,5 +51,5 @@
       rpy_offset="0 0 -0.187797428"
       mass="0.441881459418396"
-      mesh_path="package://ethercat_motor_drive/meshes"
+      mesh_path="package://moveit_config/meshes"
   />
   <xacro:create_link
@@ -58,5 +58,5 @@
       rpy_offset="0 0 0"
       mass="0.441881459418396"
-      mesh_path="package://ethercat_motor_drive/meshes"
+      mesh_path="package://moveit_config/meshes"
   />
   <!-- base_joint fixes base_link to the environment -->

Commit message: UPDATE: stepper motor is available now

File: src/moveit_config/config/moveit_config.ros2_control.xacro (robot description, xacro)
@@ -21,6 +21,6 @@
           <plugin>ethercat_generic_plugins/EcCiA402Drive</plugin>
           <param name="alias">0</param>
-          <param name="position">0</param>
-          <param name="mode_of_operation">9</param>
+          <param name="position">1</param>
+          <param name="mode_of_operation">8</param>
           <param name="slave_config">$(find moveit_config)/driver_config/tech_driver.yaml</param>
         </ec_module>
@@ -36,6 +36,6 @@
           <plugin>ethercat_generic_plugins/EcCiA402Drive</plugin>
           <param name="alias">0</param>
-          <param name="position">1</param>
-          <param name="mode_of_operation">9</param>
+          <param name="position">2</param>
+          <param name="mode_of_operation">8</param>
           <param name="slave_config">$(find moveit_config)/driver_config/tech_driver.yaml</param>
         </ec_module>
@@ -51,6 +51,6 @@
           <plugin>ethercat_generic_plugins/EcCiA402Drive</plugin>
           <param name="alias">0</param>
-          <param name="position">2</param>
-          <param name="mode_of_operation">9</param>
+          <param name="position">3</param>
+          <param name="mode_of_operation">8</param>
           <param name="slave_config">$(find moveit_config)/driver_config/tech_driver.yaml</param>
         </ec_module>
@@ -66,10 +66,10 @@
           <plugin>ethercat_generic_plugins/EcCiA402Drive</plugin>
           <param name="alias">0</param>
-          <param name="position">3</param>
-          <param name="mode_of_operation">9</param>
+          <param name="position">4</param>
+          <param name="mode_of_operation">8</param>
           <param name="slave_config">$(find moveit_config)/driver_config/tech_driver.yaml</param>
         </ec_module>
       </joint>
-      <!-- <joint name="joint6">
+      <joint name="joint6">
         <state_interface name="position"/>
         <state_interface name="velocity"/>
@@ -79,11 +79,11 @@
         <command_interface name="reset_fault"/>
         <ec_module name="Maxon">
-          <plugin>ethercat_generic_plugins/EcCiA402Drive</plugin>
+          <plugin>ethercat_generic_plugins/WaitNeededEcCiA402Drive</plugin>
           <param name="alias">0</param>
-          <param name="position">4</param>
-          <param name="mode_of_operation">9</param>
-          <param name="slave_config">$(find moveit_config)/driver_config/tech_driver.yaml</param>
+          <param name="position">0</param>
+          <param name="mode_of_operation">8</param>
+          <param name="slave_config">$(find moveit_config)/driver_config/stepper.yaml</param>
         </ec_module>
-      </joint> -->
+      </joint>
     </ros2_control>
   </xacro:macro>

File: src/moveit_config/config/robot_description.urdf.xacro (robot description, xacro)
@@ -122,5 +122,5 @@
     <limit effort="1000.0" lower="${-pi}" upper="${pi}" velocity="2.5"/>
   </joint>
-  <joint name="joint6" type="fixed">
+  <joint name="joint6" type="prismatic">
     <parent link="link5"/>
     <child link="link6"/>
