Commit message: UPDATE：

File: src/auto_store_robot_moveit_config/config/auto_store_robot_moveit_config.ros2_control.xacro (robot description, xacro)
@@ -12,4 +12,38 @@
         <param name="calculate_dynamics">true</param>
       </hardware>
+      <joint name="joint0">
+        <state_interface name="position"/>
+        <state_interface name="velocity"/>
+        <state_interface name="effort"/>
+        <state_interface name="mode"/>
+        <command_interface name="position"/>
+        <command_interface name="velocity"/>
+        <command_interface name="reset_fault"/>
+        <command_interface name="mode"/>
+        <ec_module name="inovance">
+          <plugin>ethercat_generic_plugins/EcCiA402Drive</plugin>
+          <param name="alias">0</param>
+          <param name="position">0</param>
+          <param name="mode_of_operation">8</param>
+          <param name="slave_config">$(find auto_store_robot_moveit_config)/driver_config/tech_driver.yaml</param>
+        </ec_module>
+      </joint>
+      <joint name="joint1">
+        <state_interface name="position"/>
+        <state_interface name="velocity"/>
+        <state_interface name="effort"/>
+        <state_interface name="mode"/>
+        <command_interface name="position"/>
+        <command_interface name="velocity"/>
+        <command_interface name="reset_fault"/>
+        <command_interface name="mode"/>
+        <ec_module name="Tech">
+          <plugin>ethercat_generic_plugins/EcCiA402Drive</plugin>
+          <param name="alias">0</param>
+          <param name="position">1</param>
+          <param name="mode_of_operation">8</param>
+          <param name="slave_config">$(find auto_store_robot_moveit_config)/driver_config/tech_driver.yaml</param>
+        </ec_module>
+      </joint>
       <joint name="joint2">
         <state_interface name="position"/>
@@ -21,8 +55,8 @@
         <command_interface name="reset_fault"/>
         <command_interface name="mode"/>
-        <ec_module name="Maxon">
+        <ec_module name="Tech">
           <plugin>ethercat_generic_plugins/EcCiA402Drive</plugin>
           <param name="alias">0</param>
-          <param name="position">0</param>
+          <param name="position">2</param>
           <param name="mode_of_operation">8</param>
           <param name="slave_config">$(find auto_store_robot_moveit_config)/driver_config/tech_driver.yaml</param>
@@ -38,8 +72,8 @@
         <command_interface name="reset_fault"/>
         <command_interface name="mode"/>
-        <ec_module name="Maxon">
+        <ec_module name="Tech">
           <plugin>ethercat_generic_plugins/EcCiA402Drive</plugin>
           <param name="alias">0</param>
-          <param name="position">1</param>
+          <param name="position">3</param>
           <param name="mode_of_operation">8</param>
           <param name="slave_config">$(find auto_store_robot_moveit_config)/driver_config/tech_driver.yaml</param>
@@ -55,46 +89,12 @@
         <command_interface name="reset_fault"/>
         <command_interface name="mode"/>
-        <ec_module name="Maxon">
+        <ec_module name="Tech">
           <plugin>ethercat_generic_plugins/EcCiA402Drive</plugin>
           <param name="alias">0</param>
-          <param name="position">2</param>
+          <param name="position">4</param>
           <param name="mode_of_operation">8</param>
           <param name="slave_config">$(find auto_store_robot_moveit_config)/driver_config/tech_driver.yaml</param>
         </ec_module>
       </joint>
-      <joint name="joint5">
-        <state_interface name="position"/>
-        <state_interface name="velocity"/>
-        <state_interface name="effort"/>
-        <state_interface name="mode"/>
-        <command_interface name="position"/>
-        <command_interface name="velocity"/>
-        <command_interface name="reset_fault"/>
-        <command_interface name="mode"/>
-        <ec_module name="Maxon">
-          <plugin>ethercat_generic_plugins/EcCiA402Drive</plugin>
-          <param name="alias">0</param>
-          <param name="position">3</param>
-          <param name="mode_of_operation">8</param>
-          <param name="slave_config">$(find auto_store_robot_moveit_config)/driver_config/tech_driver.yaml</param>
-        </ec_module>
-      </joint>
-<!--      <joint name="joint6">
-        <state_interface name="position"/>
-        <state_interface name="velocity"/>
-        <state_interface name="effort"/>
-        <state_interface name="mode"/>
-        <command_interface name="position"/>
-        <command_interface name="velocity"/>
-        <command_interface name="reset_fault"/>
-        <command_interface name="mode"/>
-        <ec_module name="Maxon">
-          <plugin>ethercat_generic_plugins/WaitNeededEcCiA402Drive</plugin>
-          <param name="alias">0</param>
-          <param name="position">0</param>
-          <param name="mode_of_operation">8</param>
-          <param name="slave_config">$(find auto_store_robot_moveit_config)/driver_config/stepper.yaml</param>
-        </ec_module>
-      </joint>-->
     </ros2_control>
   </xacro:macro>

File: src/auto_store_robot_moveit_config/config/auto_store_robot_moveit_config.urdf.xacro (robot description, xacro)
@@ -3,5 +3,5 @@
   <link name="world"/>
   <xacro:include filename="$(find auto_store_robot_moveit_config)/config/auto_store_robot_moveit_config.ros2_control.xacro" />
-  <xacro:include filename="$(find auto_store_robot_moveit_config)/config/robot_description.urdf.xacro" />
+  <xacro:include filename="$(find auto_store_robot_moveit_config)/config/auto_store_robot_moveit_config.urdf" />
   <xacro:motor_drive/>
   <xacro:auto_store_manipulator/>

Commit message: TMPSAVE: ready for identify and force estimation

File: src/auto_store_robot_moveit_config/config/auto_store_robot_moveit_config.ros2_control.xacro (robot description, xacro)
@@ -8,7 +8,10 @@
         <param name="control_frequency">100</param>
       </hardware> -->
-     <hardware>
+     <!-- <hardware>
         <plugin>mock_components/GenericSystem</plugin>
         <param name="calculate_dynamics">true</param>
+      </hardware> -->
+      <hardware>
+        <plugin>gz_ros2_control/GazeboSimSystem</plugin>
       </hardware>
       <joint name="joint0">
@@ -18,5 +21,5 @@
         <state_interface name="mode"/>
         <command_interface name="position"/>
-        <command_interface name="velocity"/>
+        <!-- <command_interface name="velocity"/> -->
         <command_interface name="reset_fault"/>
         <command_interface name="mode"/>
@@ -35,5 +38,5 @@
         <state_interface name="mode"/>
         <command_interface name="position"/>
-        <command_interface name="velocity"/>
+        <!-- <command_interface name="velocity"/> -->
         <command_interface name="reset_fault"/>
         <command_interface name="mode"/>
@@ -52,5 +55,5 @@
         <state_interface name="mode"/>
         <command_interface name="position"/>
-        <command_interface name="velocity"/>
+        <!-- <command_interface name="velocity"/> -->
         <command_interface name="reset_fault"/>
         <command_interface name="mode"/>
@@ -69,5 +72,5 @@
         <state_interface name="mode"/>
         <command_interface name="position"/>
-        <command_interface name="velocity"/>
+        <!-- <command_interface name="velocity"/> -->
         <command_interface name="reset_fault"/>
         <command_interface name="mode"/>
@@ -86,5 +89,5 @@
         <state_interface name="mode"/>
         <command_interface name="position"/>
-        <command_interface name="velocity"/>
+        <!-- <command_interface name="velocity"/> -->
         <command_interface name="reset_fault"/>
         <command_interface name="mode"/>
@@ -99,3 +102,4 @@
     </ros2_control>
   </xacro:macro>
+  <xacro:motor_drive/>
 </robot>

File: src/auto_store_robot_moveit_config/config/auto_store_robot_moveit_config.urdf.xacro (robot description, xacro)
@@ -1,8 +1,5 @@
 <?xml version="1.0"?>
 <robot xmlns:xacro="http://www.ros.org/wiki/xacro" name="auto_store_robot_moveit_config">
-  <link name="world"/>
   <xacro:include filename="$(find auto_store_robot_moveit_config)/config/auto_store_robot_moveit_config.ros2_control.xacro" />
   <xacro:include filename="$(find auto_store_robot_moveit_config)/config/auto_store_robot_moveit_config.urdf" />
-  <xacro:motor_drive/>
-  <xacro:auto_store_manipulator/>
 </robot>
